Commit message: Give the car 4 visual wheels at the corners instead of 2 + caster

File: src/robots/pathfinder_robot_car/urdf/car.urdf (robot description, URDF)
Before this commit: robot pathfinder_car, 4 links, 3 joints
Links:
- removed link caster_link
- removed link wheel_left
- removed link wheel_right
- added link wheel_fl, mass 0.1; collision cylinder length=0.04 radius=0.05; visual cylinder length=0.04 radius=0.05
- added link wheel_fr, mass 0.1; collision cylinder length=0.04 radius=0.05; visual cylinder length=0.04 radius=0.05
- added link wheel_rl, mass 0.1; collision cylinder length=0.04 radius=0.05; visual cylinder length=0.04 radius=0.05
- added link wheel_rr, mass 0.1; collision cylinder length=0.04 radius=0.05; visual cylinder length=0.04 radius=0.05
Joints:
- removed joint caster_joint
- removed joint left_wheel_joint
- removed joint right_wheel_joint
- added joint fl_wheel_joint: type continuous, parent base_link, child wheel_fl, origin xyz=0.13 0.16 -0.045 rpy=0 0 0, axis 0 1 0
- added joint fr_wheel_joint: type continuous, parent base_link, child wheel_fr, origin xyz=0.13 -0.16 -0.045 rpy=0 0 0, axis 0 1 0
- added joint rl_wheel_joint: type continuous, parent base_link, child wheel_rl, origin xyz=-0.13 0.16 -0.045 rpy=0 0 0, axis 0 1 0
- added joint rr_wheel_joint: type continuous, parent base_link, child wheel_rr, origin xyz=-0.13 -0.16 -0.045 rpy=0 0 0, axis 0 1 0

File: src/robots/pathfinder_robot_car/urdf/car.urdf.xacro (robot description, xacro)
@@ -12,7 +12,5 @@
   <xacro:property name="wheel_mass"       value="0.1"/>
   <xacro:property name="wheel_separation" value="0.32"/>
-  <xacro:property name="caster_radius" value="0.025"/>
-  <xacro:property name="caster_mass"   value="0.05"/>
-  <xacro:property name="caster_x"      value="0.15"/>
+  <xacro:property name="wheelbase"        value="0.26"/>
   <material name="car_dark_blue">
     <color rgba="0.1 0.15 0.4 1.0"/>
@@ -44,5 +42,5 @@
     </inertial>
   </link>
-  <xacro:macro name="drive_wheel" params="suffix y_sign">
+  <xacro:macro name="wheel" params="suffix x_sign y_sign">
     <link name="wheel_${suffix}">
       <visual>
@@ -68,41 +66,18 @@
       </inertial>
     </link>
-    <!-- Wheels mounted at y = +-(wheel_separation/2); axis along y -->
     <joint name="${suffix}_wheel_joint" type="continuous">
       <parent link="base_link"/>
       <child link="wheel_${suffix}"/>
-      <origin xyz="0 ${y_sign * wheel_separation / 2.0} ${-base_size_z/2 + wheel_radius - 0.02}" rpy="0 0 0"/>
+      <origin
+        xyz="${x_sign * wheelbase / 2.0} ${y_sign * wheel_separation / 2.0} ${-base_size_z/2 + wheel_radius - 0.02}"
+        rpy="0 0 0"/>
       <axis xyz="0 1 0"/>
     </joint>
   </xacro:macro>
-  <xacro:drive_wheel suffix="left"  y_sign="1"/>
-  <xacro:drive_wheel suffix="right" y_sign="-1"/>
-  <link name="caster_link">
-    <visual>
-      <geometry>
-        <sphere radius="${caster_radius}"/>
-      </geometry>
-      <material name="wheel_dark_gray"/>
-    </visual>
-    <collision>
-      <geometry>
-        <sphere radius="${caster_radius}"/>
-      </geometry>
-    </collision>
-    <inertial>
-      <mass value="${caster_mass}"/>
-      <inertia
-        ixx="${2.0 * caster_mass * caster_radius * caster_radius / 5.0}"
-        iyy="${2.0 * caster_mass * caster_radius * caster_radius / 5.0}"
-        izz="${2.0 * caster_mass * caster_radius * caster_radius / 5.0}"
-        ixy="0" ixz="0" iyz="0"/>
-    </inertial>
-  </link>
-  <!-- Free-swivel passive caster at the front. Caster bottom is aligned with wheel
-       bottom (base z = -0.095) so the caster doesn't drag into the ground. -->
-  <joint name="caster_joint" type="fixed">
-    <parent link="base_link"/>
-    <child link="caster_link"/>
-    <origin xyz="${caster_x} 0 -0.07" rpy="0 0 0"/>
-  </joint>
+  <!-- Visual-only 4-wheel layout (front/rear, left/right). Gazebo physics in
+       car.sdf still treats this as a diff-drive with 2 driven wheels. -->
+  <xacro:wheel suffix="fl" x_sign="1"  y_sign="1"/>
+  <xacro:wheel suffix="fr" x_sign="1"  y_sign="-1"/>
+  <xacro:wheel suffix="rl" x_sign="-1" y_sign="1"/>
+  <xacro:wheel suffix="rr" x_sign="-1" y_sign="-1"/>
 </robot>
