Commit message: Lift car chassis 10cm above base_link and hide all robot TF frames

File: src/robots/pathfinder_robot_car/urdf/car.urdf.xacro (robot description, xacro)
@@ -23,4 +23,5 @@
   <link name="base_link">
     <visual>
+      <origin xyz="0 0 0.10"/>
       <geometry>
         <box size="${base_size_x} ${base_size_y} ${base_size_z}"/>
@@ -29,4 +30,5 @@
     </visual>
     <collision>
+      <origin xyz="0 0 0.10"/>
       <geometry>
         <box size="${base_size_x} ${base_size_y} ${base_size_z}"/>

Commit message: Align car SDF physics with the 4-wheel URDF visual and remove tilt

File: src/robots/pathfinder_robot_car/urdf/car.urdf.xacro (robot description, xacro)
@@ -21,5 +21,5 @@
   <link name="base_link">
     <visual>
-      <origin xyz="0 0 0.10"/>
+      <origin xyz="0 0 0.075"/>
       <geometry>
         <box size="${base_size_x} ${base_size_y} ${base_size_z}"/>
@@ -28,5 +28,5 @@
     </visual>
     <collision>
-      <origin xyz="0 0 0.10"/>
+      <origin xyz="0 0 0.075"/>
       <geometry>
         <box size="${base_size_x} ${base_size_y} ${base_size_z}"/>
